File: hardware/KiCad/SofTub.kicad_pcb (KiCad board)
At the start: 2 copper layers, 63.5 x 36.5 mm, 9 parts, among them U2 ESP32-S2

Commit message: Version 1.0
Parts:
- moved JP1 46.9 mm to (52.1, 71.3)
- moved Temp_In1 0.62 mm to (104.7, 70.2)
- moved Top1 0.30 mm to (57.7, 73.7)
- renumbered U2 to ESP32-S2, Temp_Out1 to locked
Connections:
- ADC1 pad 3: Net-(ADC1-SCL) -> SCL
- ADC1 pad 4: Net-(ADC1-SDA) -> SDA
- ADC1 pad 8: Net-(ADC1-A0) -> Temp_in
- ADC1 pad 9: Net-(ADC1-A1) -> Temp_out
- Debug1 pad 1: Net-(ADC1-A0) -> Temp_out
- Debug1 pad 2: Net-(ADC1-A1) -> Temp_in
- Debug1 pad 3: Net-(ADC1-SDA) -> Net-(ADC1-A2)
- Debug1 pad 4: Net-(ADC1-SCL) -> unconnected-(Debug1-Pin_4-Pad4)
- Debug1 pad 5: Net-(ADC1-A2) -> unconnected-(Debug1-Pin_5-Pad5)
- ESP32-S2 pad 1: Net-(ADC1-A1) -> unconnected-(ESP32-S2-PA02_A0_D0-Pad1)
- ESP32-S2 pad 2: Net-(ADC1-A1) -> Temp_out
- ESP32-S2 pad 3: Net-(ADC1-A0) -> Temp_in
- ESP32-S2 pad 5: Net-(ADC1-SDA) -> SDA
- ESP32-S2 pad 6: Net-(ADC1-SCL) -> SCL
- Temp_In1 pad 2: Net-(ADC1-A0) -> Temp_in
- locked pad 2: Net-(ADC1-A1) -> Temp_out
Routing:
- net Net-(ADC1-A1): track 83.3 -> 0.00 mm
- net Temp_out: track 0.00 -> 80.8 mm
- net Net-(ADC1-A0): track 79.4 -> 0.00 mm
- net Temp_in: track 0.00 -> 75.9 mm
- net Net-(ADC1-SCL): track 52.6 -> 0.00 mm
- net Net-(ADC1-SDA): track 51.5 -> 0.00 mm
- net Net-(ADC1-A2): track 54.7 -> 88.5 mm
- net SDA: track 0.00 -> 33.6 mm
- net SCL: track 0.00 -> 31.2 mm
- net +5V: track 72.0 -> 101.3 mm
- net Net-(Top1-Pin_3): track 21.7 -> 50.1 mm
- net +3.3V: track 72.6 -> 86.4 mm, vias 0 -> 1
- net Net-(ESP32-S2-PA5_A9_D9_MISO): track 29.1 -> 42.3 mm
- net Net-(Top1-Pin_2): track 28.6 -> 40.6 mm
- net Net-(ESP32-S2-PA6_A10_D10_MOSI): track 32.2 -> 42.1 mm
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Other:
- board text added: "3.3"
- board text added: "5v"
- board text added: "A2"
- board text added: "ADS1115"
- board text added: "Adafruit 1085"
- board text added: "Adafruit 5325"
- board text added: "Adafruit 757"
- board text added: "BSS138"
- board text added: "Gnd"
- board text added: "RX"
- board text added: "Softub WiFi Controller https://github.com/steve1066d/softub-wifi"
- board text added: "TX"
- board text added: "Tin"
- board text added: "Tout"
- board text added: "v1.1"
- board text removed: "SoftTub Wireless Controller Steve Devore steve1066d@yahoo.com"
